Commit message: add apriltag instead of press button function

File: coover_base/autolabor_description/urdf/autolabor.urdf (robot description, URDF)
Before this commit: robot autolabor, 6 links, 5 joints
Links:
- added link link_0; visual box size=0.02 0.02 0.01
- added link right_camera_link; visual box size=0.035 0.035 0.015
Joints:
- added joint link_0_joint: type fixed, parent base_link, child link_0, origin xyz=-0.08 -0.165 1.14 rpy=0 0 0
- added joint right_camera_link_joint: type fixed, parent base_link, child right_camera_link, origin xyz=-0.23 -0.07 1.16 rpy=0 0 0
