Commit message: update campusrover arm mini config

File: campusrover_arm/campusrover_arm_description/urdf/campusrover_arm.urdf (robot description, URDF)
Before this commit: robot campusrover_arm, 7 links, 6 joints
Links:
- removed link link_0
- removed link link_1
- removed link link_2
- removed link link_3
- removed link link_4
- removed link link_5
- removed link link_6
- added link arm_link_1; collision mesh filename=package://campusrover_arm_description/meshes/arm_link_1.stl scale=0.001 0.001 0.001; visual mesh filename=package://campusrover_arm_description/meshes/arm_link_1.stl scale=0.001 0.001 0.001
- added link arm_link_2; collision mesh filename=package://campusrover_arm_description/meshes/arm_link_2.stl scale=0.001 0.001 0.001; visual mesh filename=package://campusrover_arm_description/meshes/arm_link_2.stl scale=0.001 0.001 0.001
- added link arm_link_3; collision mesh filename=package://campusrover_arm_description/meshes/arm_link_3.stl scale=0.001 0.001 0.001; visual mesh filename=package://campusrover_arm_description/meshes/arm_link_3.stl scale=0.001 0.001 0.001
- added link arm_link_4; collision mesh filename=package://campusrover_arm_description/meshes/arm_link_4.stl scale=0.001 0.001 0.001; visual mesh filename=package://campusrover_arm_description/meshes/arm_link_4.stl scale=0.001 0.001 0.001
- added link arm_link_5; collision mesh filename=package://campusrover_arm_description/meshes/arm_link_5.stl scale=0.001 0.001 0.001; visual mesh filename=package://campusrover_arm_description/meshes/arm_link_5.stl scale=0.001 0.001 0.001
- added link arm_link_6; collision box size=0.001 0.001 0.001; visual box size=0.001 0.001 0.001
Joints:
- removed joint joint_0
- joint joint_1: child link_2 -> arm_link_2; parent link_1 -> arm_link_1
- joint joint_2: child link_3 -> arm_link_3; limit lower=-1.708 upper=1.708 effort=1000.0 velocity=1.0 -> lower=-1.57 upper=1.57 effort=1000.0 velocity=1.0; origin xyz=0 0 0.0415 rpy=0 0 0 -> xyz=0 0 0.026 rpy=0 0 0; parent link_2 -> arm_link_2
- joint joint_3: child link_4 -> arm_link_4; limit lower=-0.1 upper=3.14 effort=1000.0 velocity=1.0 -> lower=-1.57 upper=1.57 effort=1000.0 velocity=1.0; origin xyz=0.043 0 0.174 rpy=0 0 0 -> xyz=0.00 0 0.1595 rpy=0 0 0; parent link_3 -> arm_link_3
- joint joint_4: child link_5 -> arm_link_5; origin xyz=0.0099 0 0.1415 rpy=0 0 0 -> xyz=0.0675 0 0.0 rpy=0 0 0; parent link_4 -> arm_link_4
- joint joint_5: child link_6 -> arm_link_6; origin xyz=0 0 0.048 rpy=0 -1.57 0 -> xyz=0.0405 0 0 rpy=0 -1.57 0; parent link_5 -> arm_link_5

File: campusrover_base/campusrover_description/urdf/campusrover.urdf (robot description, URDF)
Before this commit: robot campusrover, 9 links, 8 joints
Links:
- removed link link_0
- added link arm_link_1; visual box size=0.02 0.02 0.01
Joints:
- joint link_0_joint: child link_0 -> arm_link_1
