Commit message: updata urdf & path following.cpp

File: campusrover_base/campusrover_description/urdf/campusrover.urdf (robot description, URDF)
Before this commit: robot campusrover, 8 links, 7 joints
Joints:
- joint link_0_joint: origin xyz=-0.08 -0.165 1.14 rpy=0 0 0 -> xyz=0.027 -0.17 1.1223 rpy=0 0 0
- joint right_camera_link_joint: origin xyz=-0.23 -0.07 1.16 rpy=0 0 0 -> xyz=-0.15 -0.035 1.244 rpy=0 0 0

Commit message: update campus rover arm

File: campusrover_base/campusrover_description/urdf/campusrover.urdf (robot description, URDF)
Before this commit: robot campusrover, 8 links, 7 joints
Joints:
- joint link_0_joint: origin xyz=0.027 -0.17 1.1223 rpy=0 0 0 -> xyz=0.0 -0.245 0.89 rpy=1.57 0 0
- joint right_camera_link_joint: origin xyz=-0.15 -0.035 1.244 rpy=0 0 0 -> xyz=0.0 -0.295 0.99 rpy=0 0 0

Commit message: update elevator package

File: campusrover_base/campusrover_description/urdf/campusrover.urdf (robot description, URDF)
Before this commit: robot campusrover, 8 links, 7 joints
Joints:
- joint link_0_joint: origin xyz=0.0 -0.245 0.89 rpy=1.57 0 0 -> xyz=-0.05 -0.275 0.88 rpy=1.57 0 0
- joint right_camera_link_joint: origin xyz=0.0 -0.295 0.99 rpy=0 0 0 -> xyz=-0.05 -0.315 0.985 rpy=0 0 0

Commit message: update button recognition & add image mux

File: campusrover_base/campusrover_description/urdf/campusrover.urdf (robot description, URDF)
Before this commit: robot campusrover, 8 links, 7 joints
Links:
- added link left_camera_link; visual box size=0.035 0.035 0.015
Joints:
- added joint left_camera_link_joint: type fixed, parent base_link, child left_camera_link, origin xyz=-0.1 -0.34 0.985 rpy=0 0 -1.57

Commit message: update elevator path following for global path using

File: campusrover_base/campusrover_description/urdf/campusrover.urdf (robot description, URDF)
Before this commit: robot campusrover, 9 links, 8 joints
Joints:
- joint left_camera_link_joint: origin xyz=-0.1 -0.34 0.985 rpy=0 0 -1.57 -> xyz=0.0 -0.23 1.075 rpy=0 0 -1.57
- joint link_0_joint: origin xyz=-0.05 -0.275 0.88 rpy=1.57 0 0 -> xyz=-0.05 -0.275 0.995 rpy=1.57 0 0
- joint right_camera_link_joint: origin xyz=-0.05 -0.315 0.985 rpy=0 0 0 -> xyz=-0.05 -0.315 0.93 rpy=0 0 0

Commit message: update from campusrober_base to campusrober_base v1.1

File: campusrover_base/campusrover_description/urdf/campusrover.urdf (robot description, URDF)
Before this commit: robot campusrover, 9 links, 8 joints
Links:
- removed link left_camera_link
- removed link velodyne
- removed link wit_imu_link
- removed link ydlidar_link
- added link ydlidar_back_link; visual cylinder length=0.01 radius=0.01
- added link ydlidar_front_link; visual cylinder length=0.01 radius=0.01
Joints:
- removed joint left_camera_link_joint
- removed joint velodyne_joint
- removed joint wit_imu_link_joint
- removed joint ydlidar_link_joint
- added joint ydlidar_back_link_joint: type fixed, parent base_link, child ydlidar_back_link, origin xyz=-0.51 0 0.14 rpy=0 0 3.1415
- added joint ydlidar_front_link_joint: type fixed, parent base_link, child ydlidar_front_link, origin xyz=0.12 0 0.125 rpy=0 0 0
- joint link_0_joint: origin xyz=-0.05 -0.275 0.995 rpy=1.57 0 0 -> xyz=-0.05 -0.275 0.995 rpy=0 0 0
- joint right_camera_link_joint: origin xyz=-0.05 -0.315 0.93 rpy=0 0 0 -> xyz=-0.027 -0.09 0.0227 rpy=0 0 0; parent base_link -> arm_link_1
